Commit message: fix mesh path
Signed-off-by: Takagi, Isamu <isamu.takagi@tier4.jp>

File: models/autoware_sample_platform_launch/description/vehicle/urdf/vehicle.xacro (robot description, xacro)
@@ -8,5 +8,5 @@
       <origin xyz="${vehicle_info['/**']['ros__parameters']['wheel_base']/2.0} 0 0" rpy="${pi/2.0} 0 ${pi}"/>
       <geometry>
-        <mesh filename="package://autoware_sample_platform_launch/mesh/lexus.dae" scale="1 1 1"/>
+        <mesh filename="package://autoware_sample_platform_launch/description/vehicle/meshes/lexus.dae" scale="1 1 1"/>
       </geometry>
     </visual>
