Commit message: move files
Signed-off-by: Takagi, Isamu <isamu.takagi@tier4.jp>

File: models/autoware_sample_platform_launch/description/platform/urdf/platform.xacro (robot description, xacro)
@@ -2,4 +2,4 @@
 <robot name="vehicle" xmlns:xacro="http://ros.org/wiki/xacro">
   <xacro:include filename="$(find autoware_sample_platform_launch)/description/vehicle/urdf/vehicle.xacro"/>
-  <xacro:include filename="$(find autoware_sample_platform_launch)/description/sensors/default/urdf/sensors.xacro"/>
+  <xacro:include filename="$(find autoware_sample_platform_launch)/description/sensing/urdf/sensing.xacro"/>
 </robot>

File: models/autoware_sample_platform_launch/description/sensing/urdf/sensor_kit.xacro (robot description, xacro)
@@ -3,9 +3,9 @@
   <xacro:macro name="sensor_kit_macro" params="parent x y z roll pitch yaw">
     <xacro:include filename="$(find velodyne_description)/urdf/VLP-16.urdf.xacro"/>
-    <xacro:include filename="$(find sample_sensor_kit_description)/sensor/vls/urdf/VLS-128.urdf.xacro"/>
-    <xacro:include filename="$(find sample_sensor_kit_description)/sensor/camera/urdf/monocular_camera.xacro"/>
-    <xacro:include filename="$(find sample_sensor_kit_description)/sensor/imu/urdf/imu.xacro"/>
+    <xacro:include filename="$(find autoware_sample_platform_launch)/description/sensors/vls/urdf/VLS-128.urdf.xacro"/>
+    <xacro:include filename="$(find autoware_sample_platform_launch)/description/sensors/camera/urdf/monocular_camera.xacro"/>
+    <xacro:include filename="$(find autoware_sample_platform_launch)/description/sensors/imu/urdf/imu.xacro"/>
     <xacro:arg name="gpu" default="false"/>
-    <xacro:arg name="config_dir" default="$(find sample_sensor_kit_description)/config"/>
+    <xacro:arg name="config_dir" default="$(find autoware_sample_platform_launch)/config"/>
     <joint name="sensor_kit_base_link_joint" type="fixed">
       <origin rpy="${roll} ${pitch} ${yaw}" xyz="${x} ${y} ${z}"/>

File: models/autoware_sample_platform_launch/description/sensors/vls/urdf/VLS-128.urdf.xacro (robot description, xacro)
@@ -26,10 +26,10 @@
       <visual>
         <geometry>
-          <mesh filename="package://sample_sensor_kit_description/sensor/vls/meshes/VLS128_base_1.dae"/>
+          <mesh filename="package://autoware_sample_platform_launch/description/sensors/vls/meshes/VLS128_base_1.dae"/>
         </geometry>
       </visual>
       <visual>
         <geometry>
-          <mesh filename="package://sample_sensor_kit_description/sensor/vls/meshes/VLS128_base_2.dae"/>
+          <mesh filename="package://autoware_sample_platform_launch/description/sensors/vls/meshes/VLS128_base_2.dae"/>
         </geometry>
       </visual>
@@ -55,5 +55,5 @@
         <origin xyz="0 0 -0.06611"/>
         <geometry>
-          <mesh filename="package://sample_sensor_kit_description/sensor/vls/meshes/VLS128_scan.dae"/>
+          <mesh filename="package://autoware_sample_platform_launch/description/sensors/vls/meshes/VLS128_scan.dae"/>
         </geometry>
       </visual>
